File: H750_Core_v0.0/Connectors.sch (KiCad schematic (older format))
At the start: 6 parts, among them J1 JTAG, J2 DFU_CONN, U4 DF9-51P-1V_LEFT, U5 ESDALC6V1W5, U6 DF9-51P-1V_RIGHT

Commit message: PCB layout finished
Connections:
- net 3V3_VDD: now also U4.32 (Pin_32), U4.33 (Pin_33); no longer U4.43 (Pin_43), U4.44 (Pin_44)
- net 5V: now also U4.37 (Pin_37), U4.38 (Pin_38); no longer U4.48 (Pin_48), U4.49 (Pin_49)
- net BOOT0: now also U4.44 (Pin_44); no longer U6.45 (Pin_45)
- net GND: now also U4.34 (Pin_34), U4.35 (Pin_35), U4.36 (Pin_36), U6.1 (Pin_1), U6.2 (Pin_2), U6.32 (Pin_32), U6.51 (Pin_51); no longer U4.45 (Pin_45), U4.46 (Pin_46), U4.47 (Pin_47), U6.20 (Pin_20), U6.48 (Pin_48), U6.49 (Pin_49)
- net PA10: now also U6.47 (Pin_47); no longer U6.4 (Pin_4)
- net PA11: now also U6.48 (Pin_48); no longer U6.3 (Pin_3)
- net PA12: now also U6.49 (Pin_49); no longer U6.2 (Pin_2)
- net PA13: now also U6.50 (Pin_50); no longer U6.1 (Pin_1)
- net PA14: now also U6.15 (Pin_15); no longer U6.26 (Pin_26)
- net PA15: now also U6.14 (Pin_14); no longer U6.27 (Pin_27)
- net PA8: now also U6.45 (Pin_45); no longer U6.6 (Pin_6)
- net PA9: now also U6.46 (Pin_46); no longer U6.5 (Pin_5)
- net PB0: now also U4.27 (Pin_27); no longer U4.28 (Pin_28)
- net PB1: now also U4.26 (Pin_26); no longer U4.29 (Pin_29)
- net PB10: now also U6.26 (Pin_26); no longer U4.42 (Pin_42)
- net PB11: now also U6.27 (Pin_27); no longer U6.25 (Pin_25)
- net PB12: now also U6.28 (Pin_28); no longer U6.24 (Pin_24)
- net PB13: now also U6.29 (Pin_29); no longer U6.23 (Pin_23)
- net PB14: now also U6.30 (Pin_30); no longer U6.22 (Pin_22)
- net PB15: now also U6.31 (Pin_31); no longer U6.21 (Pin_21)
- net PB2: now also U6.25 (Pin_25); no longer U4.30 (Pin_30)
- net PB3: now also U4.49 (Pin_49); no longer U6.40 (Pin_40)
- net PB4: now also U4.48 (Pin_48); no longer U6.41 (Pin_41)
- net PB5: now also U4.47 (Pin_47); no longer U6.42 (Pin_42)
- net PB6: now also U4.46 (Pin_46); no longer U6.43 (Pin_43)
- net PB7: now also U4.45 (Pin_45); no longer U6.44 (Pin_44)
- net PB8: now also U4.43 (Pin_43); no longer U6.46 (Pin_46)
- net PB9: now also U4.42 (Pin_42); no longer U6.47 (Pin_47)
- net PC10: now also U6.13 (Pin_13); no longer U6.28 (Pin_28)
- net PC11: now also U6.12 (Pin_12); no longer U6.29 (Pin_29)
- net PC12: now also U6.11 (Pin_11); no longer U6.30 (Pin_30)
- net PC4: now also U4.29 (Pin_29); no longer U4.26 (Pin_26)
- net PC5: now also U4.28 (Pin_28); no longer U4.27 (Pin_27)
- net PC6: now also U6.41 (Pin_41); no longer U6.11 (Pin_11)
- net PC7: now also U6.42 (Pin_42); no longer U6.10 (Pin_10)
- net PC8: now also U6.43 (Pin_43); no longer U6.9 (Pin_9)
- net PC9: now also U6.44 (Pin_44); no longer U6.8 (Pin_8)
- net PD0: now also U6.10 (Pin_10); no longer U6.32 (Pin_32)
- net PD1: now also U6.9 (Pin_9); no longer U6.33 (Pin_33)
- net PD10: now also U6.35 (Pin_35); no longer U6.17 (Pin_17)
- net PD11: now also U6.36 (Pin_36); no longer U6.16 (Pin_16)
- net PD12: now also U6.37 (Pin_37); no longer U6.15 (Pin_15)
- net PD13: now also U6.38 (Pin_38); no longer U6.14 (Pin_14)
- net PD14: now also U6.39 (Pin_39); no longer U6.13 (Pin_13)
- net PD15: now also U6.40 (Pin_40); no longer U6.12 (Pin_12)
- net PD2: now also U6.5 (Pin_5); no longer U6.34 (Pin_34)
- net PD3: now also U6.6 (Pin_6); no longer U6.35 (Pin_35)
- net PD4: now also U6.7 (Pin_7); no longer U6.36 (Pin_36)
- net PD5: now also U6.8 (Pin_8); no longer U6.37 (Pin_37)
- net PD6: now also U4.51 (Pin_51); no longer U6.38 (Pin_38)
- net PD7: now also U4.50 (Pin_50); no longer U6.39 (Pin_39)
- net PD8: now also U6.33 (Pin_33); no longer U6.19 (Pin_19)
- net PD9: now also U6.34 (Pin_34); no longer U6.18 (Pin_18)
- net PE0: now also U4.41 (Pin_41); no longer U4.51 (Pin_51)
- net PE1: now also U4.40 (Pin_40); no longer U4.50 (Pin_50)
- net PE10: now also U6.21 (Pin_21); no longer U4.35 (Pin_35)
- net PE11: now also U6.16 (Pin_16); no longer U4.36 (Pin_36)
- net PE12: now also U6.17 (Pin_17); no longer U4.37 (Pin_37)
- net PE13: now also U6.18 (Pin_18); no longer U4.38 (Pin_38)
- net PE14: now also U6.19 (Pin_19); no longer U4.39 (Pin_39)
- net PE15: now also U6.20 (Pin_20); no longer U4.40 (Pin_40)
- net PE7: now also U6.24 (Pin_24); no longer U4.32 (Pin_32)
- net PE8: now also U6.23 (Pin_23); no longer U4.33 (Pin_33)
- net PE9: now also U6.22 (Pin_22); no longer U4.34 (Pin_34)
- net VIN: now also U6.3 (Pin_3), U6.4 (Pin_4); no longer U6.50 (Pin_50), U6.51 (Pin_51)
- net VREFP renamed VREFP_Ext
- no-connect marks 6 -> 5

Commit message: 修改编程接口
Parts:
- removed J1: JTAG, Connector_PinSocket_2.54mm:PinSocket_2x05_P2.54mm_Vertical, symbol Connector_Generic:Conn_02x05_Odd_Even
- removed R4: 10K, Resistor_SMD:R_0603_1608Metric, symbol Device:R_Small
- added J1: DFU_CONN, Connector_PinHeader_2.54mm:PinHeader_1x05_P2.54mm_Vertical, symbol Connector:Conn_01x05_Male
- J2: footprint Connector_PinSocket_2.54mm:PinSocket_1x04_P2.54mm_Vertical -> Connector_JST:JST_EH_B5B-EH-A_1x05_P2.50mm_Vertical; symbol Connector:Conn_01x04_Male -> Connector:Conn_01x05_Male
Connections:
- net 3V3_VDD: now also J2.5 (Pin_5), J1.5 (Pin_5); no longer J2.4 (Pin_4)
- net GND: now also J2.3 (Pin_3), J1.3 (Pin_3); no longer J2.2 (Pin_2)
- net PE11: now also U6.20 (Pin_20); no longer U6.16 (Pin_16)
- net PE12: now also U6.19 (Pin_19); no longer U6.17 (Pin_17)
- net PE14: now also U6.17 (Pin_17); no longer U6.19 (Pin_19)
- net PE15: now also U6.16 (Pin_16); no longer U6.20 (Pin_20)
- net SWCLK: now also J2.4 (Pin_4), J1.4 (Pin_4); no longer J2.3 (Pin_3)
- net SWDIO: now also J2.2 (Pin_2), J1.2 (Pin_2); no longer J2.1 (Pin_1)
- net SWO: now also J2.1 (Pin_1), J1.1 (Pin_1)
- net T_JTDI: no longer names the net of U5.5
Changed lines of the file:
@@
 EESchema Schematic File Version 4
-LIBS:H750_Core-cache
 EELAYER 30 0
 EELAYER END
@@
 	1    0    0    -1
 $EndComp
-Text HLabel 8700 6450 2    50   BiDi ~ 0
-SWDIO
-Text HLabel 8700 6550 2    50   BiDi ~ 0
-SWCLK
-Text HLabel 8700 6750 2    50   BiDi ~ 0
-T_JTDI
-Text HLabel 8700 6650 2    50   BiDi ~ 0
-SWO
 Text HLabel 8550 3050 2    50   BiDi ~ 0
 BOOT0
@@
 Text Label 8300 4750 2    50   ~ 0
 PB0
-Text Label 10000 4300 0    50   ~ 0
+Text Label 10000 3900 0    50   ~ 0
 PE15
-Text Label 10000 4200 0    50   ~ 0
+Text Label 10000 4000 0    50   ~ 0
 PE14
 Text Label 10000 4100 0    50   ~ 0
 PE13
-Text Label 10000 4000 0    50   ~ 0
+Text Label 10000 4200 0    50   ~ 0
 PE12
-Text Label 10000 3900 0    50   ~ 0
+Text Label 10000 4300 0    50   ~ 0
 PE11
 Text Label 10000 4400 0    50   ~ 0
@@
 PE7
 Wire Wire Line
+	10000 3900 10400 3900
+Wire Wire Line
+	10000 4000 10400 4000
+Wire Wire Line
+	10000 4100 10400 4100
+Wire Wire Line
+	10000 4200 10400 4200
+Wire Wire Line
 	10000 4300 10400 4300
-Wire Wire Line
-	10000 4200 10400 4200
-Wire Wire Line
-	10000 4100 10400 4100
-Wire Wire Line
-	10000 4000 10400 4000
-Wire Wire Line
-	10000 3900 10400 3900
 Wire Wire Line
 	10000 4400 10400 4400
@@
 Wire Wire Line
 	8550 3050 7900 3050
-Text HLabel 8700 6850 2    50   BiDi ~ 0
-NRST
-Wire Wire Line
-	8550 6450 8700 6450
-Wire Wire Line
-	8550 6550 8700 6550
-Wire Wire Line
-	8550 6650 8700 6650
-Wire Wire Line
-	8550 6750 8700 6750
-Wire Wire Line
-	8550 6850 8700 6850
-Text GLabel 7550 6450 0    50   BiDi ~ 0
-3V3_VDD
-Wire Wire Line
-	7550 6450 8050 6450
-$Comp
-L power:GND #PWR013
-U 1 1 5D97C451
-P 7550 6650
-F 0 "#PWR013" H 7550 6400 50  0001 C CNN
-F 1 "GND" V 7555 6522 50  0000 R CNN
-F 2 "" H 7550 6650 50  0001 C CNN
-F 3 "" H 7550 6650 50  0001 C CNN
-	1    7550 6650
-	0    1    1    0
-$EndComp
-Wire Wire Line
-	7550 6650 7800 6650
-Wire Wire Line
-	8050 6550 7800 6550
-Wire Wire Line
-	7800 6550 7800 6650
-Connection ~ 7800 6650
-Wire Wire Line
-	7800 6650 8050 6650
-$Comp
-L power:GND #PWR012
-U 1 1 5D996424
-P 7300 6850
-F 0 "#PWR012" H 7300 6600 50  0001 C CNN
-F 1 "GND" V 7305 6722 50  0000 R CNN
-F 2 "" H 7300 6850 50  0001 C CNN
-F 3 "" H 7300 6850 50  0001 C CNN
-	1    7300 6850
-	0    1    1    0
-$EndComp
-$Comp
-L Device:R_Small R4
-U 1 1 5D997327
-P 7650 6850
-F 0 "R4" V 7454 6850 50  0000 C CNN
-F 1 "10K" V 7545 6850 50  0000 C CNN
-F 2 "Resistor_SMD:R_0603_1608Metric" H 7650 6850 50  0001 C CNN
-F 3 "~" H 7650 6850 50  0001 C CNN
-	1    7650 6850
-	0    1    1    0
-$EndComp
-Wire Wire Line
-	7550 6850 7300 6850
-Wire Wire Line
-	7750 6850 8050 6850
-NoConn ~ 8050 6750
-$Comp
-L Connector_Generic:Conn_02x05_Odd_Even J1
-U 1 1 5D9C1307
-P 8250 6650
-F 0 "J1" H 8300 7067 50  0000 C CNN
-F 1 "JTAG" H 8300 6976 50  0000 C CNN
-F 2 "Connector_PinSocket_2.54mm:PinSocket_2x05_P2.54mm_Vertical" H 8250 6650 50  0001 C CNN
-F 3 "~" H 8250 6650 50  0001 C CNN
-	1    8250 6650
-	1    0    0    -1
-$EndComp
-$Comp
-L Connector:Conn_01x04_Male J2
+$Comp
+L Connector:Conn_01x05_Male J2
 U 1 1 5D9C3EC6
 P 9700 6600
-F 0 "J2" H 9808 6881 50  0000 C CNN
-F 1 "DFU_CONN" H 9808 6790 50  0000 C CNN
-F 2 "Connector_PinSocket_2.54mm:PinSocket_1x04_P2.54mm_Vertical" H 9700 6600 50  0001 C CNN
+F 0 "J2" H 9800 7050 50  0000 C CNN
+F 1 "DFU_CONN" H 9800 6950 50  0000 C CNN
+F 2 "Connector_JST:JST_EH_B5B-EH-A_1x05_P2.50mm_Vertical" H 9700 6600 50  0001 C CNN
 F 3 "~" H 9700 6600 50  0001 C CNN
 	1    9700 6600
@@
 Text HLabel 7750 8100 0    50   BiDi ~ 0
 SWCLK
-Text HLabel 7750 7700 0    50   BiDi ~ 0
-T_JTDI
 Text HLabel 7750 7850 0    50   BiDi ~ 0
 SWO
@@
 Wire Wire Line
 	10150 2400 10400 2400
+Text HLabel 10100 6400 2    50   BiDi ~ 0
+SWO
+Wire Wire Line
+	10100 6400 9900 6400
+NoConn ~ 7750 7700
+$Comp
+L Connector:Conn_01x05_Male J1
+U 1 1 5E4AEDC5
+P 8300 6600
+F 0 "J1" H 8400 7050 50  0000 C CNN
+F 1 "DFU_CONN" H 8400 6950 50  0000 C CNN
+F 2 "Connector_PinHeader_2.54mm:PinHeader_1x05_P2.54mm_Vertical" H 8300 6600 50  0001 C CNN
+F 3 "~" H 8300 6600 50  0001 C CNN
+	1    8300 6600
+	1    0    0    -1
+$EndComp
+Text HLabel 8700 6500 2    50   BiDi ~ 0
+SWDIO
+Text HLabel 8700 6700 2    50   BiDi ~ 0
+SWCLK
+$Comp
+L power:GND #PWR060
+U 1 1 5E4AEDCD
+P 9050 6600
+F 0 "#PWR060" H 9050 6350 50  0001 C CNN
+F 1 "GND" V 9055 6472 50  0000 R CNN
+F 2 "" H 9050 6600 50  0001 C CNN
+F 3 "" H 9050 6600 50  0001 C CNN
+	1    9050 6600
+	0    -1   -1   0
+$EndComp
+Text GLabel 8700 7000 2    50   BiDi ~ 0
+3V3_VDD
+Wire Wire Line
+	9050 6600 8500 6600
+Wire Wire Line
+	8700 7000 8700 6800
+Wire Wire Line
+	8700 6800 8500 6800
+Wire Wire Line
+	8700 6700 8500 6700
+Wire Wire Line
+	8700 6500 8500 6500
+Text HLabel 8700 6400 2    50   BiDi ~ 0
+SWO
+Wire Wire Line
+	8700 6400 8500 6400
 Wire Bus Line
 	2450 2150 2450 4550
