File: H750_Core_v0.0/Ethernet.sch (KiCad schematic (older format))
At the start: 40 parts, among them U10 RJ45, U7 LAN8742A-CZ-TR, U8 USBLC6-4, U9 H1102NL, Y3 NX2016SA 25MHz

Commit message: PCB layout finished
Parts:
- JP17: footprint Resistor_SMD:R_0603_1608Metric -> H750_Core:JP
Changed lines of the file:
@@
 F 0 "JP17" H 3500 5245 50  0000 C CNN
 F 1 "Jumper_2_Bridged" H 3500 5154 50  0000 C CNN
-F 2 "Resistor_SMD:R_0603_1608Metric" H 3500 5050 50  0001 C CNN
+F 2 "H750_Core:JP" H 3500 5050 50  0001 C CNN
 F 3 "~" H 3500 5050 50  0001 C CNN
 	1    3500 5050
