File: H750_Core_v0.0/MCU_Power.sch (KiCad schematic (older format))
At the start: 21 parts, among them U1 750VB_3Parts

Commit message: PCB layout finished
Parts:
- JP19, JP20, JP21: footprint Resistor_SMD:R_0603_1608Metric -> H750_Core:JP
Connections:
- net VREFP: no longer JP19.1 (A)
- new net VREFP_Ext: JP19.1 (A)
Changed lines of the file:
@@
 F 0 "JP20" V 3404 2058 50  0000 L CNN
 F 1 "Jumper_2_Bridged" V 3495 2058 50  0000 L CNN
-F 2 "Resistor_SMD:R_0603_1608Metric" H 3450 2000 50  0001 C CNN
+F 2 "H750_Core:JP" H 3450 2000 50  0001 C CNN
 F 3 "~" H 3450 2000 50  0001 C CNN
 	1    3450 2000
@@
 F 0 "JP21" H 7200 5945 50  0000 C CNN
 F 1 "Jumper_2_Bridged" H 7200 5854 50  0000 C CNN
-F 2 "Resistor_SMD:R_0603_1608Metric" H 7200 5750 50  0001 C CNN
+F 2 "H750_Core:JP" H 7200 5750 50  0001 C CNN
 F 3 "~" H 7200 5750 50  0001 C CNN
 	1    7200 5750
@@
 	7450 6200 7000 6200
 Text GLabel 2250 3550 0    50   BiDi ~ 0
-VREFP
+VREFP_Ext
 $Comp
 L Jumper:Jumper_2_Open JP19
@@
 F 0 "JP19" H 2500 3785 50  0000 C CNN
 F 1 "Jumper_2_Open" H 2500 3694 50  0000 C CNN
-F 2 "Resistor_SMD:R_0603_1608Metric" H 2500 3550 50  0001 C CNN
+F 2 "H750_Core:JP" H 2500 3550 50  0001 C CNN
 F 3 "~" H 2500 3550 50  0001 C CNN
 	1    2500 3550
