File: H750_Core_v0.0/Main_Power.sch (KiCad schematic (older format))
At the start: 21 parts, among them U11 TPS786_5V, U12 TPS786_3V3

Commit message: PCB layout finished
Parts:
- JP18: footprint Resistor_SMD:R_0603_1608Metric -> H750_Core:JP
Changed lines of the file:
@@
 F 0 "JP18" H 7100 2945 50  0000 C CNN
 F 1 "Jumper_2_Bridged" H 7100 2854 50  0000 C CNN
-F 2 "Resistor_SMD:R_0603_1608Metric" H 7100 2750 50  0001 C CNN
+F 2 "H750_Core:JP" H 7100 2750 50  0001 C CNN
 F 3 "~" H 7100 2750 50  0001 C CNN
 	1    7100 2750

Commit message: 修改编程接口
Parts:
- removed R28: 25K, Resistor_SMD:R_0603_1608Metric, symbol Device:R_Small
- removed R29: 30.1K, Resistor_SMD:R_0603_1608Metric, symbol Device:R_Small
- removed R30: 79K, Resistor_SMD:R_0603_1608Metric, symbol Device:R_Small
- removed R31: 52.3K, Resistor_SMD:R_0603_1608Metric, symbol Device:R_Small
- added C46, C47: 10nF, Capacitor_SMD:C_0603_1608Metric, symbol Device:C
- C25: value 10uF -> 2.2uF
- C26: value 4.7uF -> 2.2uF
Connections:
- net GND: now also C23.2, C24.2, C46.2, C47.2
- net at U11.5 (NR/FB): now also C46.1; no longer C23.2
- net at U12.5 (NR/FB): now also C47.1; no longer C24.2
Other:
- moved on the sheet: C20, C22, C24, C26, R27, U12
